Commit message: Added parameters for port name, baud rate and dynamixel id

File: dynamixel_ros_control/config/ros2_control_test_config.xacro (robot description, xacro)
@@ -1,16 +1,16 @@
 <?xml version="1.0"?>
 <robot xmlns:xacro="http://www.ros.org/wiki/xacro">
-    <xacro:macro name="ros2_control_test_config">
+    <xacro:macro name="ros2_control_test_config" params="port_name baud_rate id">
         <ros2_control name="hardware_interface" type="system">
             <hardware>
                 <plugin>dynamixel_ros_control/DynamixelHardwareInterface</plugin>
                 <param name="debug">true</param>
-                <param name="port_name">/dev/ttyUSB0</param>
-                <param name="baud_rate">57600</param>
+                <param name="port_name">${port_name}</param>
+                <param name="baud_rate">${baud_rate}</param>
                 <param name="torque_on_startup">true</param>
                 <param name="torque_off_on_shutdown">false</param>
             </hardware>
             <joint name="joint_1">
-                <param name="id">1</param>
+                <param name="id">${id}</param>
                 <param name="position_control_mode">extended_position</param>
                 <command_interface name="position"/>

File: dynamixel_ros_control/config/test_robot.urdf.xacro (robot description, xacro)
@@ -10,4 +10,4 @@
     <link name="link_1"/>
     <xacro:include filename="$(find dynamixel_ros_control)/config/ros2_control_test_config.xacro" />
-    <xacro:ros2_control_test_config/>
+    <xacro:ros2_control_test_config port_name="$(arg port_name)" baud_rate="$(arg baud_rate)" id="$(arg id)"/>
 </robot>

Commit message: Added transmission interface

File: dynamixel_ros_control/config/ros2_control_test_config.xacro (robot description, xacro)
@@ -10,5 +10,5 @@
                 <param name="torque_on_startup">true</param>
                 <param name="torque_off_on_shutdown">true</param>
-                <param name="reboot_on_hardware_error">true</param>
+                <param name="reboot_on_hardware_error">false</param>
             </hardware>
             <joint name="joint_1">
@@ -23,4 +23,12 @@
                 <state_interface name="effort"/>
             </joint>
+            <transmission name="transmission1">
+                <plugin>transmission_interface/SimpleTransmission</plugin>
+                <actuator name="actuator_1" role="actuator_1"/>
+                <joint name="joint_1" role="joint_1">
+                    <mechanical_reduction>2.0</mechanical_reduction>
+                    <offset>0.0</offset>
+                </joint>
+            </transmission>
         </ros2_control>
     </xacro:macro>
